File: pcb/v1/ssc01.kicad_pcb (KiCad board)
At the start: 2 copper layers, 100 x 80 mm, 31 parts, among them J1 UART, J2 USB_B_Mini, SW1 Reset, U1 74HCT04, U2 MC68B50, U3 74LS32, U4 Z80CPU, U5 SST39SF040, U6 62256, Y1 7.3728Hz

Commit message: continue layout
Parts:
- moved R5 23.9 mm to (113.9, 37.0)
- moved C4 3.45 mm to (49.9, 84.1)
- moved U1 3.45 mm to (60.6, 83.8)
- moved R3 1.19 mm to (117.0, 49.4)
- moved R4 1.04 mm to (117.0, 37.0)
- moved C3 0.45 mm to (92.5, 52.2)
Routing:
- net VCC: track 277.7 -> 432.0 mm, vias 0 -> 3
- net /BANK1: track 0.00 -> 111.8 mm, vias 0 -> 2
- net /BANK2: track 0.00 -> 106.7 mm, vias 0 -> 2
- net /BANK0: track 0.00 -> 101.8 mm, vias 0 -> 1
- net Net-(U1-Pad2): track 0.00 -> 93.7 mm, vias 0 -> 3
- net /~WR: track 0.00 -> 89.5 mm, vias 0 -> 5
- net /D0: track 26.3 -> 115.1 mm, vias 0 -> 6
- net /D1: track 26.3 -> 110.0 mm, vias 0 -> 5
- net /CLOCK: track 65.5 -> 148.3 mm, vias 1 -> 2
- net /~MEM_RD: track 0.00 -> 82.5 mm, vias 0 -> 4
- net /A7: track 0.00 -> 77.0 mm, vias 0 -> 5
- net /A0: track 11.1 -> 83.1 mm, vias 0 -> 6
- net /A6: track 11.1 -> 82.3 mm, vias 0 -> 5
- net Net-(U3-Pad1): track 0.00 -> 70.2 mm, vias 0 -> 1
- net /A10: track 0.00 -> 69.7 mm, vias 0 -> 4
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- added copper zone on B.Cu, net GND
- added copper zone on F.Cu, net GND

Commit message: continue layout
Parts:
- D1: footprint LED_THT:LED_D5.0mm -> LED_SMD:LED_1206_3216Metric
- moved D1 2.74 mm to (93.6, 92.2), turned to 0 degrees
Routing:
- net Net-(U3-Pad1): track 70.2 -> 82.4 mm
- net /A0: track 83.1 -> 72.9 mm, vias 6 -> 2
- net /D1: track 110.0 -> 104.4 mm, vias 5 -> 2
- net VCC: track 432.0 -> 426.7 mm
- net /A8: track 49.8 -> 45.6 mm, vias 4 -> 2
- net /A6: track 82.3 -> 78.8 mm, vias 5 -> 3
- net /D6: track 91.7 -> 88.7 mm, vias 6 -> 4
- net /D3: track 105.3 -> 102.6 mm, vias 5 -> 4
- net /A7: track 77.0 -> 74.6 mm, vias 5 -> 3
- net /A5: track 53.0 -> 51.1 mm
- net /A11: track 70.4 -> 68.7 mm, vias 4 -> 3
- net /D7: track 107.1 -> 105.5 mm
- net /A9: track 51.0 -> 49.4 mm, vias 5 -> 4
- net Net-(U1-Pad4): track 55.0 -> 53.5 mm
- net /~INT: track 101.9 -> 100.5 mm, vias 2 -> 1
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Other:
- board text added: "Ilya Strukov's Single-board Computer 1 rev. A"

Commit message: complete layout
Parts:
- D1: value POWER_LED -> POWER
Other:
- board text added: "0"
- board text added: "1"
- board text added: "2"
- board text added: "ROM bank"
Changed lines of the file:
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@@
   (general
     (thickness 1.6)
-    (drawings 9)
+    (drawings 15)
     (tracks 776)
     (zones 0)
@@
     (pad_to_mask_clearance 0.051)
     (solder_mask_min_width 0.25)
-    (aux_axis_origin 0 0)
+    (aux_axis_origin 20 20)
     (visible_elements FFFFFF7F)
     (pcbplotparams
@@
       (effects (font (size 1 1) (thickness 0.15)))
     )
-    (fp_text value 0.1uF (at -2 -0.5 180) (layer F.SilkS)
+    (fp_text value 0.1uF (at 1.18 -2.16 270) (layer F.SilkS)
       (effects (font (size 1 1) (thickness 0.15)))
     )
@@
     (descr "C, Disc series, Radial, pin pitch=2.50mm, , diameter*width=3.8*2.6mm^2, Capacitor, http://www.vishay.com/docs/45233/krseries.pdf")
     (tags "C Disc series Radial pin pitch 2.50mm  diameter 3.8mm width 2.6mm Capacitor")
-    (fp_text reference C4 (at 1.25 -2.55 90) (layer F.SilkS)
-      (effects (font (size 1 1) (thickness 0.15)))
-    )
-    (fp_text value 0.1uF (at 1.25 2.55 90) (layer F.Fab)
+    (fp_text reference C4 (at 1.25 -2.55 90) (layer F.SilkS) hide
+      (effects (font (size 1 1) (thickness 0.15)))
+    )
+    (fp_text value 0.1uF (at 1.18 -2.51 270) (layer F.SilkS)
       (effects (font (size 1 1) (thickness 0.15)))
     )
@@
     (descr "C, Disc series, Radial, pin pitch=2.50mm, , diameter*width=3.8*2.6mm^2, Capacitor, http://www.vishay.com/docs/45233/krseries.pdf")
     (tags "C Disc series Radial pin pitch 2.50mm  diameter 3.8mm width 2.6mm Capacitor")
-    (fp_text reference C5 (at 4.5 0) (layer F.SilkS)
-      (effects (font (size 1 1) (thickness 0.15)))
-    )
-    (fp_text value 0.1uF (at 1.25 2.55 270) (layer F.Fab)
+    (fp_text reference C5 (at 4.5 0) (layer F.SilkS) hide
+      (effects (font (size 1 1) (thickness 0.15)))
+    )
+    (fp_text value 0.1uF (at 1.19 -2.35 270) (layer F.SilkS)
       (effects (font (size 1 1) (thickness 0.15)))
     )
@@
     (descr "C, Disc series, Radial, pin pitch=2.50mm, , diameter*width=3.8*2.6mm^2, Capacitor, http://www.vishay.com/docs/45233/krseries.pdf")
     (tags "C Disc series Radial pin pitch 2.50mm  diameter 3.8mm width 2.6mm Capacitor")
-    (fp_text reference C7 (at 4.25 0) (layer F.SilkS)
-      (effects (font (size 1 1) (thickness 0.15)))
-    )
-    (fp_text value 0.1uF (at 1.25 2.55 270) (layer F.Fab)
+    (fp_text reference C7 (at 4.25 0) (layer F.SilkS) hide
+      (effects (font (size 1 1) (thickness 0.15)))
+    )
+    (fp_text value 0.1uF (at 1.23 -2.22 270) (layer F.SilkS)
       (effects (font (size 1 1) (thickness 0.15)))
     )
@@
     (descr "C, Disc series, Radial, pin pitch=2.50mm, , diameter*width=3.8*2.6mm^2, Capacitor, http://www.vishay.com/docs/45233/krseries.pdf")
     (tags "C Disc series Radial pin pitch 2.50mm  diameter 3.8mm width 2.6mm Capacitor")
-    (fp_text reference C8 (at 1.25 -2.55 90) (layer F.SilkS)
-      (effects (font (size 1 1) (thickness 0.15)))
-    )
-    (fp_text value 0.1uF (at 1.25 2.55 90) (layer F.Fab)
+    (fp_text reference C8 (at 1.25 -2.55 90) (layer F.SilkS) hide
+      (effects (font (size 1 1) (thickness 0.15)))
+    )
+    (fp_text value 0.1uF (at 1.27 -2.38 90) (layer F.SilkS)
       (effects (font (size 1 1) (thickness 0.15)))
     )
@@
     (tags diode)
     (attr smd)
-    (fp_text reference D1 (at 0 -1.82) (layer F.SilkS)
-      (effects (font (size 1 1) (thickness 0.15)))
-    )
-    (fp_text value POWER_LED (at 0 1.82) (layer F.Fab)
+    (fp_text reference D1 (at 0 -1.82) (layer F.SilkS) hide
+      (effects (font (size 1 1) (thickness 0.15)))
+    )
+    (fp_text value POWER (at -0.01 -2.22) (layer F.SilkS)
       (effects (font (size 1 1) (thickness 0.15)))
     )
@@
     )
   )
+  (gr_text 1 (at 94.51 80.37) (layer F.SilkS)
+    (effects (font (size 1.1 1.1) (thickness 0.15)))
+  )
+  (gr_text 0 (at 94.56 85.91) (layer F.SilkS)
+    (effects (font (size 1.1 1.1) (thickness 0.15)))
+  )
+  (gr_text 2 (at 104.26 88.32) (layer F.SilkS)
+    (effects (font (size 1.1 1.1) (thickness 0.15)))
+  )
+  (gr_text 1 (at 100.66 88.32) (layer F.SilkS)
+    (effects (font (size 1.1 1.1) (thickness 0.15)))
+  )
+  (gr_text 0 (at 96.96 88.32) (layer F.SilkS)
+    (effects (font (size 1.1 1.1) (thickness 0.15)))
+  )
+  (gr_text "ROM bank" (at 100.31 78.03) (layer F.SilkS)
+    (effects (font (size 1.1 1.1) (thickness 0.15)))
+  )
   (gr_text "Ilya Strukov's Single-board Computer 1 rev. A" (at 70.42 97.87) (layer F.SilkS)

Commit message: WIP
Parts:
- U6: footprint Package_DIP:DIP-28_W7.62mm_LongPads -> Package_DIP:DIP-28_W15.24mm_LongPads
- moved R5 48.2 mm to (90.8, 79.3)
- moved R1 15.3 mm to (25.0, 86.5)
- moved JP4 8.40 mm to (113.0, 80.5), turned to 90 degrees
- moved C5 4.25 mm to (93.2, 24.2)
- moved C3 3.81 mm to (96.2, 52.0)
- moved U2 3.51 mm to (98.8, 24.0)
- moved U6 3.25 mm to (75.0, 24.2)
- moved C4 3.10 mm to (46.8, 84.1)
- moved U1 3.10 mm to (57.5, 83.8)
- moved U5 3.00 mm to (50.0, 24.2)
- moved C7 2.75 mm to (68.5, 24.2)
- moved U4 2.25 mm to (25.5, 24.2)
- moved C6 2.00 mm to (22.2, 49.8)
- moved C8 0.50 mm to (71.7, 84.4)
- moved U3 0.50 mm to (82.7, 84.0)
Routing:
- net VCC: track 426.7 -> 2.54 mm, vias 3 -> 0
- net /BANK1: track 110.6 -> 0.00 mm, vias 1 -> 0
- net /BANK2: track 106.5 -> 0.00 mm, vias 1 -> 0
- net /BANK0: track 101.8 -> 0.00 mm, vias 1 -> 0
- net Net-(U1-Pad2): track 93.7 -> 0.00 mm, vias 3 -> 0
- net /~WR: track 89.5 -> 0.00 mm, vias 5 -> 0
- net /CLOCK: track 148.3 -> 63.3 mm
- net /~MEM_RD: track 82.4 -> 0.00 mm, vias 4 -> 0
- net Net-(U3-Pad1): track 82.4 -> 0.00 mm, vias 1 -> 0
- net /A6: track 78.8 -> 10.3 mm, vias 3 -> 0
- net /A7: track 74.6 -> 10.3 mm, vias 3 -> 0
- net /D7: track 105.5 -> 42.7 mm, vias 7 -> 0
- net /D0: track 114.0 -> 55.9 mm, vias 5 -> 2
- net Net-(U3-Pad2): track 54.2 -> 0.00 mm, vias 2 -> 0
- net Net-(U1-Pad4): track 53.5 -> 0.00 mm, vias 2 -> 0
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
Commit message: layout in progress
Routing:
- net /~INT: track 100.7 -> 0.00 mm, vias 2 -> 0
- net /A4: track 62.5 -> 10.3 mm, vias 2 -> 0
- net /A1: track 62.5 -> 10.3 mm, vias 2 -> 0
- net /A2: track 62.5 -> 10.3 mm, vias 2 -> 0
- net /A3: track 62.4 -> 10.3 mm, vias 2 -> 0
- net /A0: track 59.9 -> 10.3 mm, vias 2 -> 0
- net /A5: track 49.8 -> 10.3 mm, vias 2 -> 0
- net /A12: track 65.0 -> 30.5 mm, vias 4 -> 2
- net /D2: track 68.1 -> 36.0 mm, vias 4 -> 2
- net /D1: track 55.9 -> 26.6 mm, vias 2 -> 0
- net /D0: track 55.9 -> 26.7 mm, vias 2 -> 0
- net /~M1: track 75.1 -> 77.0 mm

Commit message: layout in progress
Parts:
- moved C6 0.27 mm to (22.5, 49.6)
Routing:
- net VCC: track 2.54 -> 307.5 mm, vias 0 -> 1
- net /~M1: track 77.0 -> 0.00 mm, vias 2 -> 0
- net /A6: track 10.3 -> 82.2 mm, vias 0 -> 3
- net /A7: track 10.3 -> 78.0 mm, vias 0 -> 2
- net /A2: track 10.3 -> 61.7 mm, vias 0 -> 1
- net /A1: track 10.3 -> 61.6 mm, vias 0 -> 1
- net /A4: track 10.3 -> 60.0 mm, vias 0 -> 1
- net /A3: track 10.3 -> 60.0 mm, vias 0 -> 1
- net /A0: track 10.3 -> 59.2 mm, vias 0 -> 1
- net /BANK1: track 0.00 -> 38.8 mm, vias 0 -> 1
- net /A12: track 30.5 -> 67.6 mm, vias 2 -> 4
- net /BANK0: track 0.00 -> 37.0 mm, vias 0 -> 1
- net /BANK2: track 0.00 -> 36.4 mm, vias 0 -> 1
- net /A5: track 10.3 -> 46.4 mm, vias 0 -> 1
- net /D5: track 52.8 -> 84.4 mm, vias 2 -> 3
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
Commit message: second take at the layout
Parts:
- moved R2 0.95 mm to (71.7, 92.2)
- moved C8 0.50 mm to (71.7, 83.9)
- moved C4 0.30 mm to (46.8, 83.8)
- moved R8 0.15 mm to (87.5, 92.2)
- moved U3 0.15 mm to (82.7, 83.8)
Routing:
- net /~INT: track 0.00 -> 113.2 mm, vias 0 -> 2
- net /~M1: track 0.00 -> 90.9 mm, vias 0 -> 3
- net /~WR: track 0.00 -> 82.0 mm, vias 0 -> 1
- net /CLOCK: track 63.3 -> 145.1 mm, vias 2 -> 4
- net Net-(U3-Pad1): track 0.00 -> 71.1 mm, vias 0 -> 1
- net /BANK1: track 38.8 -> 107.3 mm, vias 1 -> 2
- net VCC: track 307.5 -> 373.5 mm
- net /BANK2: track 36.4 -> 101.2 mm
- net /BANK0: track 37.0 -> 101.4 mm, vias 1 -> 2
- net Net-(U1-Pad4): track 0.00 -> 63.3 mm, vias 0 -> 1
- net /D1: track 57.2 -> 120.1 mm, vias 1 -> 3
- net /D0: track 56.8 -> 117.8 mm, vias 1 -> 3
- net /~MEM_WR: track 0.00 -> 60.7 mm, vias 0 -> 1
- net /~RTS: track 0.00 -> 49.9 mm, vias 0 -> 1
- net Net-(U3-Pad2): track 0.00 -> 49.4 mm, vias 0 -> 1
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
Commit message: finish second layout iteration
Routing:
- net /D0: track 117.8 -> 109.8 mm, vias 3 -> 1
- net Net-(C1-Pad1): track 37.1 -> 33.1 mm
- net /~IORQ: track 36.6 -> 34.6 mm, vias 1 -> 0
- net /A14: track 70.0 -> 68.4 mm
- net Net-(U3-Pad1): track 71.1 -> 69.8 mm, vias 1 -> 0
- net /A13: track 65.4 -> 66.8 mm, vias 4 -> 3
- net /A3: track 55.8 -> 57.0 mm
- net /A10: track 63.6 -> 63.0 mm
- net /A2: track 58.3 -> 58.9 mm
- net /MEM_SEL: track 88.3 -> 87.7 mm
- net /D4: track 106.0 -> 105.6 mm, vias 3 -> 2
Other:
- board text added: "+5V"
- board text added: "GND"
- board text added: "RTS"
- board text added: "RX"
- board text added: "TX"
