File: pcb/v1/ssc01.kicad_pcb (KiCad board)
At the start: 2 copper layers, 100 x 80 mm, 31 parts, among them J1 UART, J2 USB_B_Mini, SW1 Reset, U1 74HCT04, U2 MC68B50, U3 74LS32, U4 Z80CPU, U5 SST39SF040, U6 62256, Y1 7.3728Hz

Commit message: replace the MC68B50 footprint
Parts:
- U2: footprint Package_DIP:DIP-40_W15.24mm -> Package_DIP:DIP-24_W15.24mm_LongPads
- moved JP4 53.3 mm to (112.2, 27.2)
- moved U2 47.8 mm to (111.9, 70.0), turned to 180 degrees
- moved R5 38.8 mm to (115.9, 49.6), turned to 270 degrees
- moved J1 34.0 mm to (113.0, 21.9), turned to 270 degrees
- moved C3 21.2 mm to (115.0, 42.0)
- moved R3 20.4 mm to (101.8, 35.8), turned to 0 degrees
- moved R4 15.9 mm to (101.7, 32.6), turned to 0 degrees
Routing:
- net /~RTS: track 49.9 -> 3.98 mm, vias 1 -> 0
- net /D1: track 120.1 -> 89.0 mm, vias 3 -> 2
- net /D7: track 106.1 -> 78.6 mm, vias 3 -> 1
- net /CLOCK: track 145.1 -> 124.4 mm, vias 4 -> 2
- net /RXD: track 19.4 -> 39.7 mm
- net /A6: track 82.2 -> 98.8 mm, vias 3 -> 2
- net /D0: track 109.8 -> 93.3 mm, vias 1 -> 3
- net Net-(U1-Pad4): track 63.3 -> 77.6 mm
- net Net-(J1-Pad3): track 26.0 -> 13.3 mm
- net /D3: track 106.9 -> 94.7 mm
- net /A7: track 78.0 -> 89.8 mm, vias 2 -> 1
- net /D2: track 105.8 -> 94.3 mm
- net /D5: track 100.6 -> 90.2 mm
- net /D6: track 94.2 -> 84.2 mm
- net /D4: track 105.6 -> 95.7 mm
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Other:
- board text added: "Ilya Strukov's Single-board Computer 1 rev. B"
- board text removed: "Ilya Strukov's Single-board Computer 1 rev. A"

Commit message: move some tracks
Parts:
- moved R5 1.44 mm to (115.2, 50.9)
- moved C3 0.16 mm to (115.2, 42.0), turned to 270 degrees
Routing:
- net /MEM_SEL: track 87.7 -> 83.7 mm
- net /A10: track 63.0 -> 59.3 mm
- net /A11: track 69.1 -> 65.9 mm
- net /D2: track 94.3 -> 91.4 mm
- net /D1: track 89.0 -> 86.5 mm
- net /A13: track 66.8 -> 64.6 mm
- net /A9: track 47.5 -> 45.3 mm
- net /D0: track 93.3 -> 91.4 mm
- net /A7: track 89.8 -> 91.6 mm, vias 1 -> 2
- net /A8: track 41.1 -> 39.5 mm
- net /A0: track 77.5 -> 79.0 mm
- net /~M1: track 91.3 -> 90.1 mm
- net VCC: track 378.9 -> 377.7 mm
- net Net-(J1-Pad5): track 39.7 -> 38.6 mm
- net /D4: track 95.7 -> 94.7 mm
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