File: pcb/v1/ssc01.sch (KiCad schematic (older format))
At the start: 31 parts, among them J1 UART, J2 USB_B_Mini, SW1 Reset, U1 74HCT04, U2 MC68B50, U3 74LS32, U4 Z80CPU, U5 SST39SF040, U6 62256, Y1 7.3728Hz

Commit message: complete layout
Parts:
- D1: value POWER_LED -> POWER
Changed lines of the file:
@@
 P 2200 5340
 F 0 "D1" V 2238 5222 50  0000 R CNN
-F 1 "POWER_LED" V 2147 5222 50  0000 R CNN
+F 1 "POWER" V 2147 5222 50  0000 R CNN
 F 2 "LED_SMD:LED_1206_3216Metric" H 2200 5340 50  0001 C CNN
 F 3 "~" H 2200 5340 50  0001 C CNN

Commit message: WIP
Parts:
- U6: footprint Package_DIP:DIP-28_W7.62mm_LongPads -> Package_DIP:DIP-28_W15.24mm_LongPads
Changed lines of the file:
@@
 F 0 "U6" H 9140 2480 50  0000 C CNN
 F 1 "62256" H 8860 1600 50  0000 C CNN
-F 2 "Package_DIP:DIP-28_W7.62mm_LongPads" H 9130 2480 50  0001 C CNN
+F 2 "Package_DIP:DIP-28_W15.24mm_LongPads" H 9130 2480 50  0001 C CNN
 F 3 "" H 9130 2480 50  0001 C CNN
 	1    9130 2480

Commit message: replace the MC68B50 footprint
Parts:
- U2: footprint Package_DIP:DIP-40_W15.24mm -> Package_DIP:DIP-24_W15.24mm_LongPads
Changed lines of the file:
@@
 F 0 "U2" H 5080 6170 50  0000 C CNN
 F 1 "MC68B50" H 4720 4990 50  0000 C CNN
-F 2 "Package_DIP:DIP-40_W15.24mm" H 5140 5020 50  0001 L CNN
+F 2 "Package_DIP:DIP-24_W15.24mm_LongPads" H 5140 5020 50  0001 L CNN
 F 3 "http://pdf.datasheetcatalog.com/datasheet/motorola/MC6850.pdf" H 5090 6170 50  0001 C CNN
 	1    5090 6170
